File: ArduinoNanoBoard.kicad_pcb (KiCad board)
At the start: 2 copper layers, 6 parts, among them J1 Conn_01x15_Male, J2 Conn_01x04_Male, J3 Conn_01x10_Male

Commit message: BOPIR02 ADD FINGERPRINTS
Parts:
- added G***: LOGO, IDG_LOGO:triangulo, F.Cu at (147.3, 134.6)
- added G***: LOGO, IDG_LOGO:skulls2, F.Cu at (208.3, 116.8)

Commit message: BOPIR03 - J CONECTORS RFID AND BLUETOOTH
Parts:
- removed the G*** at (208.3, 116.8)
- added J4: Conn_01x08_Male, Connector_PinHeader_2.54mm:PinHeader_1x08_P2.54mm_Vertical, F.Cu at (177.8, 129.5)
- added J5: Conn_01x04_Male, Connector_PinHeader_2.54mm:PinHeader_1x04_P2.54mm_Vertical, F.Cu at (175.3, 94.0)
Routing:
- net Net-(A1-Pad13): track 25.4 -> 136.7 mm, vias 0 -> 2
- net Net-(A1-Pad6): track 25.4 -> 111.1 mm, vias 0 -> 2
- net GND: track 54.2 -> 130.1 mm
- net Net-(A1-Pad5): track 25.4 -> 98.7 mm, vias 0 -> 3
- net Net-(A1-Pad12): track 25.4 -> 81.0 mm, vias 0 -> 1
- net Net-(A1-Pad27): track 50.0 -> 103.5 mm
- net Net-(A1-Pad14): track 25.4 -> 77.8 mm, vias 0 -> 1
- net Net-(A1-Pad15): track 25.4 -> 76.2 mm, vias 0 -> 1
- net Net-(A1-Pad17): track 49.8 -> 90.7 mm
- net Net-(A1-Pad16): track 61.1 -> 93.7 mm, vias 0 -> 2
