File: ArduinoNanoBoard.kicad_sch (KiCad schematic)
At the start: 4 parts, among them J1 Conn_01x15_Male, J2 Conn_01x04_Male, J3 Conn_01x10_Male

Commit message: BOPIR03 - J CONECTORS RFID AND BLUETOOTH
Parts:
- added J4: Conn_01x08_Male, Connector_PinHeader_2.54mm:PinHeader_1x08_P2.54mm_Vertical, symbol Connector:Conn_01x08_Male
- added J5: Conn_01x04_Male, Connector_PinHeader_2.54mm:PinHeader_1x04_P2.54mm_Vertical, symbol Connector:Conn_01x04_Male
Connections:
- net GND: now also J4.3 (Pin_3), J5.2 (Pin_2)
- net at A1.12 (D9), J1.11 (Pin_11): now also J4.2 (Pin_2)
- net at A1.13 (D10), J1.12 (Pin_12): now also J4.8 (Pin_8)
- net at A1.14 (D11), J1.13 (Pin_13): now also J4.6 (Pin_6)
- net at A1.15 (D12), J1.14 (Pin_14): now also J4.5 (Pin_5)
- net at A1.16 (D13), J1.15 (Pin_15): now also J4.7 (Pin_7)
- net at A1.5 (D2), J1.4 (Pin_4): now also J5.3 (Pin_3)
- net at A1.6 (D3), J1.5 (Pin_5): now also J5.4 (Pin_4)
- net at A1.27 (+5V), J2.2 (Pin_2): now also J5.1 (Pin_1)
- net at A1.17 (3V3), J2.3 (Pin_3): now also J4.1 (Pin_1)
- no-connect marks 2 -> 3
